File: PCB Files/smd_single_layer/smd_board_singlelayer.brd (EAGLE design)
At the start: 40 x 50 mm, 29 parts, among them IC1 MEGA8-AI, J1 22-27-2041-04, J2 22-27-2021-02, J3 I2C, J4 I2C, Q1 16MHz, X1 22-23-2031, X2 22-23-2031, X3 22-23-2031, X4 22-23-2031, X5 87758-0216

Commit message: updated files
Routing:
- added copper zone on layer 1, net GND
- removed copper zone on layer 16, net GND
Changed lines of the file:
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@@
 <layer number="224" name="224bmp" color="25" fill="1" visible="no" active="no"/>
 <layer number="248" name="Housing" color="7" fill="1" visible="yes" active="yes"/>
-<layer number="249" name="Edge" color="7" fill="1" visible="no" active="yes"/>
+<layer number="249" name="Edge" color="7" fill="1" visible="yes" active="yes"/>
 <layer number="250" name="Descript" color="3" fill="1" visible="no" active="no"/>
 <layer number="251" name="SMDround" color="12" fill="11" visible="no" active="no"/>
-<layer number="254" name="cooling" color="7" fill="1" visible="no" active="yes"/>
+<layer number="254" name="cooling" color="7" fill="1" visible="yes" active="yes"/>
 </layers>
 <board>
@@
 <contactref element="T3" pad="E"/>
 <contactref element="T4" pad="E"/>
-<polygon width="0.4064" layer="16">
+<polygon width="0.4064" layer="1">
 <vertex x="0.9525" y="0.635"/>
-<vertex x="1.0325" y="48.925"/>
-<vertex x="39.1325" y="48.925"/>
+<vertex x="1.0325" y="49.2425"/>
+<vertex x="39.1325" y="49.2425"/>
 <vertex x="39.0525" y="0.9525"/>
 </polygon>
@@
 <wire x1="24.765" y1="16.1925" x2="25.4951" y2="16.1925" width="0.508" layer="1"/>
 <wire x1="25.4951" y1="16.1925" x2="25.5651" y2="16.2625" width="0.508" layer="1"/>
-<wire x1="35.2425" y1="32.385" x2="35.2425" y2="37.7825" width="0" layer="19" extent="1-1"/>
-<wire x1="31.75" y1="30.985" x2="35.2425" y2="32.385" width="0" layer="19" extent="1-1"/>
-<wire x1="27.6225" y1="35.2425" x2="31.75" y2="30.985" width="0" layer="19" extent="1-1"/>
-<wire x1="25.0825" y1="41.5925" x2="27.6225" y2="41.5925" width="0" layer="19" extent="1-1"/>
-<wire x1="29.21" y1="24.895" x2="31.75" y2="30.985" width="0" layer="19" extent="1-1"/>
-<wire x1="25.5651" y1="17.8625" x2="29.21" y2="24.895" width="0" layer="19" extent="1-1"/>
-<wire x1="27.305" y1="14.7925" x2="25.5651" y2="16.2625" width="0" layer="19" extent="1-1"/>
-<wire x1="29.21" y1="14.7925" x2="27.305" y2="14.7925" width="0" layer="19" extent="1-1"/>
-<wire x1="16.9799" y1="17.0625" x2="24.13" y2="17.4625" width="0" layer="19" extent="1-1"/>
-<wire x1="14.2875" y1="13.84" x2="16.9799" y2="17.0625" width="0" layer="19" extent="1-1"/>
-<wire x1="12.195" y1="13.0175" x2="14.2875" y2="13.84" width="0" layer="19" extent="1-1"/>
-<wire x1="11.7475" y1="10.16" x2="12.195" y2="13.0175" width="0" layer="19" extent="1-1"/>
-<wire x1="5.3975" y1="16.8275" x2="12.195" y2="13.0175" width="0" layer="19" extent="1-1"/>
-<wire x1="15.11" y1="44.1325" x2="25.0825" y2="41.5925" width="0" layer="19" extent="1-1"/>
-<wire x1="10.6475" y1="43.5" x2="15.11" y2="44.1325" width="0" layer="19" extent="1-1"/>
-<wire x1="6.3475" y1="37.9525" x2="10.6475" y2="43.5" width="0" layer="19" extent="1-1"/>
 </signal>
 <signal name="+5V">
@@
 <wire x1="26.3525" y1="9.8425" x2="37.1475" y2="9.8425" width="0.508" layer="1"/>
 <wire x1="37.1475" y1="9.8425" x2="37.7825" y2="10.4775" width="0.508" layer="1"/>
-<wire x1="24.0725" y1="12.44" x2="24.0725" y2="13.1699" width="0" layer="19" extent="16-16"/>
+<wire x1="24.0725" y1="12.44" x2="24.0725" y2="13.1699" width="0" layer="19" extent="1-1"/>
 </signal>
 <signal name="N$14">
